File: Eagle Project/HCSR04/HCSR04.sch (EAGLE design)
At the start: 37 parts, among them J1 PIC_ICSP_6_PIN, T1 BC847

Commit message: PCB done
Parts:
- removed C10: (no value), adafruit:C-US025-024X044
- removed C2: (no value), adafruit:C-US050-050X075
- added C14, C15, C16, C17, C18: 150n, adafruit:C-US025-024X044
- added C19: 1u2, adafruit:C-US025-024X044
- added IC1: 4053N, 40xx:4053N
- added JP1: (no value), adafruit:PINHD-1X1
- added Q1: BC857ALT1SMD, transistor-pnp:BC857ALT1SMD
- added Q2: 12MHz, crystal:CRYSTALHC33U-V
- added R21: 1K, adafruit:R-US_0204/2V
- added SG1: EFBRD22C41, buzzer:EFBRD22C41
- added U$3: MAX232_TIN, max232ti_n:MAX232_TIN
- C1: value (none) -> 10n; device rcl:C-EU050-045X075 -> adafruit:C-US025-024X044
- C11, C12: value (none) -> 22p
- C13, C7: value (none) -> 1u2
- C3, C4: value (none) -> 1n
- C5: value (none) -> 12p
- C6, C9: value (none) -> 10n
- C8: value (none) -> 150n
- R1, R10, R6: value (none) -> 10k
- R11, R9: value (none) -> 120k
- R12, R13, R4: value (none) -> 1k
- R14, R18, R19, R20: value (none) -> 10K
- R15: value (none) -> 3K9
- R16: value (none) -> 75K
- R17: value (none) -> 3M3
- R2: value (none) -> 62k
- R3: value (none) -> 2k2
- R5: value (none) -> 18k
- R7: value (none) -> 75k
- R8: value (none) -> 4k53
Connections:
- removed net GND2: C10.2
- removed net V+: C10.1
- new net 1.0V: IC1P.VEE
- new net N$12: R21.1, U$2.PA3(T0)
- new net N$22: C15.1, U$3.C1+
- new net N$26: C16.1, U$3.C2+
- new net N$27: C17.2, U$3.VS-
- new net N$28: C14.1, C18.2, Q1.C, U$3.VCC
- new net N$29: C15.2, U$3.C1-
- new net N$30: C16.2, U$3.C2-
- new net N$31: Q1.B, R21.2
- new net N$32: IC1A.X0, R1.1
- new net N$33: U$2.PA7(ICP), U$3.T1IN
- new net N$34: U$2.PB2(INT0), U$3.T2IN
- new net N$35: IC1A.X, SG1.1
- new net N$36: IC1A.X1, U$3.T1OUT
- new net N$37: IC1A.Y, SG1.2
- new net N$38: IC1A.A, IC1A.B, JP1.1
- net 3.3V: now also C14.2, C17.1, C19.1, IC1A.Y0, IC1P.GND, U$3.GND
- net 5V: now also C18.1, C19.2, IC1P.VCC, Q1.E, R12.2, U$3.VS+
- net N$1: no longer C2.1
- net N$15: now also IC1A.Y1, U$3.T2OUT; no longer R12.2
- net N$2: no longer C2.2
- net N$23: now also Q2.2
- net N$24: now also Q2.1
